File: main.sch (EAGLE design)
At the start: 25 parts, among them J1 9V-1294-2PIN, J2 20020316-H021B01LF:TERM_BLOCK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, M1 IRLML2502TRPBF:SOT-23-3, U1 LP2985-50DBVR:SOT-23-5, U2 MMA2240KEG:SOIC-16W, U3 BAS4002A-RPP:SOT-143, U4 LTC6992CS6-1:SOT-23-6

Commit message: added distributor and distributor p/n attributes to parts
Parts:
- C1: DISTRIBUTOR (none) -> Digi-key; DISTRIBUTOR_PN (none) -> 399-10429-1-ND
- C10, C2, C6, C8, C9: DISTRIBUTOR (none) -> Digi-key; DISTRIBUTOR_PN (none) -> 1276-1007-1-ND
- C3: DISTRIBUTOR (none) -> Digi-key; DISTRIBUTOR_PN (none) -> 1276-1066-1-ND
- C4, C7: DISTRIBUTOR (none) -> Digi-key; DISTRIBUTOR_PN (none) -> 311-1136-1-ND
- C5: DISTRIBUTOR (none) -> Digi-key; DISTRIBUTOR_PN (none) -> 445-1420-1-ND
- R1, R5: DISTRIBUTOR (none) -> Digi-key; DISTRIBUTOR_PN (none) -> 311-1.0KARCT-ND
- R2: DISTRIBUTOR (none) -> Digi-key; DISTRIBUTOR_PN (none) -> 311-1.00MCRCT-ND
- R3: DISTRIBUTOR (none) -> Digi-key; DISTRIBUTOR_PN (none) -> 311-100KCRCT-ND
- R4: DISTRIBUTOR (none) -> Digi-key; DISTRIBUTOR_PN (none) -> 311-680ARCT-ND
- R6: DISTRIBUTOR (none) -> Digi-key; DISTRIBUTOR_PN (none) -> CPA25Q10.0CT-ND
